File: ml621_charger.kicad_pcb (KiCad board)
At the start: 2 copper layers, 22.5 x 12.7 mm, 15 parts, among them J1 USB_B_Micro, Q1 BSS138, U1 ATtiny10-TS, U2 AMS1117-3.3

Commit message: Fix charger
Parts:
- removed REF**: Logo_WM, Symbol:Logo_WM
- moved C1 3.99 mm to (125.1, 96.4)
- turned R5 to 180 degrees
Connections:
- BT1 pad 2: GND -> Net-(BT1-Pad2)
- Q1 pad 2: V_REG -> GND
- Q1 pad 3: Net-(Q1-Pad3) -> Net-(BT1-Pad2)
- R5 pad 1: Net-(Q1-Pad3) -> VBAT
- R5 pad 2: VBAT -> V_REG
Routing:
- net V_REG: track 14.3 -> 20.5 mm
- net Net-(BT1-Pad2): track 0.00 -> 5.83 mm, vias 0 -> 1
- net Net-(Q1-Pad1): track 17.4 -> 14.7 mm
- net GND: track 5.44 -> 7.65 mm
- net Net-(Q1-Pad3): track 1.80 -> 0.00 mm
Other:
- board text added: "v3.0.1 08/02/20"
- board text removed: "v3.0.0 05/24/20"
